Commit message: panda reach plate

File: custom_envs/envs/robots/panda_plate.urdf (robot description, URDF)
Before this commit: robot panda, 13 links, 12 joints
Links:
- removed link panda_grasptarget
- removed link panda_leftfinger
- removed link panda_rightfinger
- link panda_hand: geometry collision cylinder length=0.02 radius=0.15; visual cylinder length=0.02 radius=0.15
Joints:
- removed joint panda_finger_joint1
- removed joint panda_finger_joint2
- removed joint panda_grasptarget_hand
